File: dwm1001_adapter/v1.brd (EAGLE design)
At the start: 36.5 x 27.9 mm, 39 parts

Commit message: -updates to schematic and board
Parts:
- removed R7, R8: (no value), rcl:R0603
- removed RXD, TXD: (no value), RMSlib:CHIPLED_0603
- moved RST 3.81 mm to (31.8, 8.89), turned to 270 degrees
- moved TP2 1.66 mm to (1.78, 6.99)
- moved RESET 1.27 mm to (33.0, 26.7)
- moved TP3 1.27 mm to (8.89, 26.7)
- moved R4 1.27 mm to (33.0, 16.5)
- moved SFDLED 1.27 mm to (27.9, 16.5)
- moved TP11 1.27 mm to (19.1, 16.5)
- moved J1 1.27 mm to (20.3, 3.81)
- moved J2 1.27 mm to (11.4, 6.35)
- moved R1 1.27 mm to (33.0, 24.1)
- moved R2 1.27 mm to (33.0, 21.6)
- moved R5 1.27 mm to (33.0, 19.1)
- moved R6 1.27 mm to (2.16, 11.4)
- moved RXLED 1.27 mm to (27.9, 24.1)
- moved RXOKLED 1.27 mm to (27.9, 19.1)
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Connections:
- removed net N$10: R7.2, RXD.C
- removed net N$11: R8.2, TXD.C
- net GND: no longer R7.1, R8.1
- net RXD: no longer RXD.A
- net TXD: no longer TXD.A
Routing:
- net /RESET: track 58.5 -> 45.4 mm
- net N$11: track 3.48 -> 0.00 mm
- net N$10: track 3.48 -> 0.00 mm
- net SCL: track 19.1 -> 21.6 mm
- net READY: track 16.5 -> 19.1 mm
- net SDA: track 23.3 -> 25.8 mm
- net BT_WAKE_UP: track 27.9 -> 29.3 mm
- net RXD: track 31.3 -> 30.1 mm
- net TXD: track 29.1 -> 28.2 mm
Other:
- board size 36.5 x 27.9 mm -> 36.5 x 29.2 mm
- board text added: "BT_WAKE"
- board text removed: "BT_WAKE_UP"
- board text removed: "DWM1001"

Commit message: - updated board and schematic
Parts:
- removed J2: (no value), SparkFun-Connectors:MOLEX-1X4
- removed RST: SPST, SparkFun-Switches:TACTILE_SWITCH_PTH_6.0MM
- removed TP1, TP2: TEST-POINT2, SparkFun-Connectors:PAD.02X.02
- removed TP10, TP11, TP12, TP13, TP14, TP15, TP16, TP5, TP6, TP7, TP8, TP9: (no value), SparkFun-Connectors:TP_15TH
- removed TP17: MISO, SparkFun-Connectors:TP_15TH
- removed TP18: MOSI, SparkFun-Connectors:TP_15TH
- removed TP19: SCK, SparkFun-Connectors:TP_15TH
- removed TP20: SS, SparkFun-Connectors:TP_15TH
- removed TP3: SWD_CLK, SparkFun-Connectors:TP_15TH
- removed TP4: SWD_SIO, SparkFun-Connectors:TP_15TH
- added PROG: (no value), DC_LOAD_AU:1X04
Connections:
- removed net /SSEL: TP20.P$1, U$1.P29
- removed net MISO: TP17.P$1, U$1.P26
- removed net MOSI: TP18.P$1, U$1.P27
- removed net N$13: TP5.P$1, U$1.P25
- removed net N$14: TP4.P$1, U$1.P3
- removed net N$15: TP6.P$1, U$1.P5
- removed net N$16: TP7.P$1, U$1.P4
- removed net N$17: TP8.P$1, U$1.P6
- removed net N$18: TP9.P$1, U$1.P17
- removed net N$19: TP10.P$1, U$1.P7
- removed net N$20: TP11.P$1, U$1.P23
- removed net N$21: TP12.P$1, U$1.P8
- removed net N$22: TP13.P$1, U$1.P16
- removed net N$23: TP14.P$1, U$1.P13
- removed net N$24: TP15.P$1, U$1.P10
- removed net N$25: TP16.P$1, U$1.P9
- removed net N$5: TP3.P$1, U$1.P2
- removed net SCK: TP19.P$1, U$1.P28
- new net SWD_CLK: PROG.2, U$1.P2
- new net SWD_SIO: PROG.3, U$1.P3
- net /RESET: no longer RST.3
- net GND: now also PROG.4; no longer J2.1, RESET.1, TP2.P$1
- net RXD: no longer J2.3
- net TXD: no longer J2.2
- net VCC: now also PROG.1, RESET.1; no longer J2.4, RST.1, TP1.P$1
Routing:
- net SWD_CLK: track 0.00 -> 27.7 mm, vias 0 -> 1
- net VCC: track 0.00 -> 27.6 mm, vias 3 -> 4
- net SWD_SIO: track 0.00 -> 25.2 mm, vias 0 -> 1
- net RXD: track 30.1 -> 10.2 mm, vias 1 -> 0
- net TXD: track 28.2 -> 10.7 mm
- net N$23: track 7.65 -> 0.00 mm
- net N$25: track 5.54 -> 0.00 mm
- net N$19: track 5.20 -> 0.00 mm
- net N$18: track 5.13 -> 0.00 mm
- net N$14: track 5.12 -> 0.00 mm
- net N$15: track 5.10 -> 0.00 mm
- net SCK: track 4.99 -> 0.00 mm
- net MISO: track 4.98 -> 0.00 mm
- net N$20: track 4.95 -> 0.00 mm
- net N$22: track 3.97 -> 0.00 mm
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Other:
- board text added: "DWM1001 Breakout rev2 E. Hunckler 2018"
- board text removed: "DWM1001 Breakout rev1 E. Hunckler 2018"
