File: dwm1001_adapter/v1.sch (EAGLE design)
At the start: 39 parts

Commit message: -updates to schematic and board
Parts:
- removed R7, R8: (no value), rcl:R-US_R0603
- removed RXD, TXD: (no value), RMSlib:LEDCHIPLED_0603
Connections:
- removed net N$10: R7.2, RXD.C
- removed net N$11: R8.2, TXD.C
- net GND: no longer R7.1, R8.1
- net RXD: no longer RXD.A
- net TXD: no longer TXD.A
Changed lines of the file:
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@@
 <?xml version="1.0" encoding="utf-8"?>
 <!DOCTYPE eagle SYSTEM "eagle.dtd">
-<eagle version="8.2.1">
+<eagle version="8.4.2">
 <drawing>
 <settings>
 <setting alwaysvectorfont="no"/>
+<setting keepoldvectorfont="yes"/>
 <setting verticaltext="up"/>
 </settings>
 <grid distance="0.1" unitdist="inch" unit="inch" style="lines" multiple="1" display="no" altdistance="0.01" altunitdist="inch" altunit="inch"/>
 <layers>
-<layer number="1" name="Top" color="4" fill="1" visible="yes" active="no"/>
-<layer number="16" name="Bottom" color="1" fill="1" visible="yes" active="no"/>
-<layer number="17" name="Pads" color="2" fill="1" visible="yes" active="no"/>
-<layer number="18" name="Vias" color="2" fill="1" visible="yes" active="no"/>
-<layer number="19" name="Unrouted" color="6" fill="1" visible="yes" active="no"/>
-<layer number="20" name="Dimension" color="15" fill="1" visible="yes" active="no"/>
-<layer number="21" name="tPlace" color="7" fill="1" visible="yes" active="no"/>
-<layer number="22" name="bPlace" color="7" fill="1" visible="yes" active="no"/>
-<layer number="23" name="tOrigins" color="15" fill="1" visible="yes" active="no"/>
-<layer number="24" name="bOrigins" color="15" fill="1" visible="yes" active="no"/>
-<layer number="25" name="tNames" color="7" fill="1" visible="yes" active="no"/>
-<layer number="26" name="bNames" color="7" fill="1" visible="yes" active="no"/>
-<layer number="27" name="tValues" color="7" fill="1" visible="yes" active="no"/>
-<layer number="28" name="bValues" color="7" fill="1" visible="yes" active="no"/>
+<layer number="1" name="Top" color="4" fill="1" visible="no" active="no"/>
+<layer number="16" name="Bottom" color="1" fill="1" visible="no" active="no"/>
+<layer number="17" name="Pads" color="2" fill="1" visible="no" active="no"/>
+<layer number="18" name="Vias" color="2" fill="1" visible="no" active="no"/>
+<layer number="19" name="Unrouted" color="6" fill="1" visible="no" active="no"/>
+<layer number="20" name="Dimension" color="15" fill="1" visible="no" active="no"/>
+<layer number="21" name="tPlace" color="7" fill="1" visible="no" active="no"/>
+<layer number="22" name="bPlace" color="7" fill="1" visible="no" active="no"/>
+<layer number="23" name="tOrigins" color="15" fill="1" visible="no" active="no"/>
+<layer number="24" name="bOrigins" color="15" fill="1" visible="no" active="no"/>
+<layer number="25" name="tNames" color="7" fill="1" visible="no" active="no"/>
+<layer number="26" name="bNames" color="7" fill="1" visible="no" active="no"/>
+<layer number="27" name="tValues" color="7" fill="1" visible="no" active="no"/>
+<layer number="28" name="bValues" color="7" fill="1" visible="no" active="no"/>
 <layer number="29" name="tStop" color="7" fill="3" visible="no" active="no"/>
 <layer number="30" name="bStop" color="7" fill="6" visible="no" active="no"/>
@@
 <layer number="35" name="tGlue" color="7" fill="4" visible="no" active="no"/>
 <layer number="36" name="bGlue" color="7" fill="5" visible="no" active="no"/>
-<layer number="37" name="tTest" color="7" fill="1" visible="yes" active="no"/>
-<layer number="38" name="bTest" color="7" fill="1" visible="yes" active="no"/>
+<layer number="37" name="tTest" color="7" fill="1" visible="no" active="no"/>
+<layer number="38" name="bTest" color="7" fill="1" visible="no" active="no"/>
 <layer number="39" name="tKeepout" color="4" fill="11" visible="no" active="no"/>
 <layer number="40" name="bKeepout" color="1" fill="11" visible="no" active="no"/>
@@
 <layer number="44" name="Drills" color="7" fill="1" visible="no" active="no"/>
 <layer number="45" name="Holes" color="7" fill="1" visible="no" active="no"/>
-<layer number="46" name="Milling" color="3" fill="1" visible="yes" active="no"/>
-<layer number="47" name="Measures" color="7" fill="1" visible="yes" active="no"/>
-<layer number="48" name="Document" color="7" fill="1" visible="yes" active="no"/>
-<layer number="49" name="Reference" color="7" fill="1" visible="yes" active="no"/>
-<layer number="50" name="dxf" color="7" fill="1" visible="yes" active="no"/>
-<layer number="51" name="tDocu" color="7" fill="1" visible="yes" active="no"/>
-<layer number="52" name="bDocu" color="7" fill="1" visible="yes" active="no"/>
-<layer number="53" name="tGND_GNDA" color="7" fill="9" visible="yes" active="no"/>
-<layer number="54" name="bGND_GNDA" color="1" fill="9" visible="yes" active="no"/>
-<layer number="56" name="wert" color="7" fill="1" visible="yes" active="no"/>
-<layer number="57" name="tCAD" color="7" fill="1" visible="yes" active="no"/>
-<layer number="59" name="tCarbon" color="7" fill="1" visible="yes" active="no"/>
-<layer number="60" name="bCarbon" color="7" fill="1" visible="yes" active="no"/>
+<layer number="46" name="Milling" color="3" fill="1" visible="no" active="no"/>
+<layer number="47" name="Measures" color="7" fill="1" visible="no" active="no"/>
+<layer number="48" name="Document" color="7" fill="1" visible="no" active="no"/>
+<layer number="49" name="Reference" color="7" fill="1" visible="no" active="no"/>
+<layer number="50" name="dxf" color="7" fill="1" visible="no" active="no"/>
+<layer number="51" name="tDocu" color="7" fill="1" visible="no" active="no"/>
+<layer number="52" name="bDocu" color="7" fill="1" visible="no" active="no"/>
+<layer number="53" name="tGND_GNDA" color="7" fill="9" visible="no" active="no"/>
+<layer number="54" name="bGND_GNDA" color="1" fill="9" visible="no" active="no"/>
+<layer number="56" name="wert" color="7" fill="1" visible="no" active="no"/>
+<layer number="57" name="tCAD" color="7" fill="1" visible="no" active="no"/>
+<layer number="59" name="tCarbon" color="7" fill="1" visible="no" active="no"/>
+<layer number="60" name="bCarbon" color="7" fill="1" visible="no" active="no"/>
 <layer number="90" name="Modules" color="5" fill="1" visible="yes" active="yes"/>
 <layer number="91" name="Nets" color="2" fill="1" visible="yes" active="yes"/>
@@
 <part name="VCCLED" library="RMSlib" deviceset="LED" device="CHIPLED_0603"/>
 <part name="R6" library="rcl" deviceset="R-US_" device="R0603"/>
-<part name="RXD" library="RMSlib" deviceset="LED" device="CHIPLED_0603"/>
-<part name="R7" library="rcl" deviceset="R-US_" device="R0603"/>
-<part name="TXD" library="RMSlib" deviceset="LED" device="CHIPLED_0603"/>
-<part name="R8" library="rcl" deviceset="R-US_" device="R0603"/>
 <part name="P+5" library="supply1" library_urn="urn:adsk.eagle:library:371" deviceset="VCC" device=""/>
 <part name="J1" library="SparkFun-Connectors" library_urn="urn:adsk.eagle:library:513" deviceset="CONN_05X2" device="RAF"/>
@@
 <instance part="VCCLED" gate="G$1" x="22.86" y="99.06"/>
 <instance part="R6" gate="G$1" x="22.86" y="86.36" rot="R90"/>
-<instance part="RXD" gate="G$1" x="38.1" y="99.06"/>
-<instance part="R7" gate="G$1" x="38.1" y="86.36" rot="R90"/>
-<instance part="TXD" gate="G$1" x="30.48" y="99.06"/>
-<instance part="R8" gate="G$1" x="30.48" y="86.36" rot="R90"/>
 <instance part="P+5" gate="VCC" x="22.86" y="116.84"/>
 <instance part="J1" gate="G$1" x="132.08" y="170.18"/>
@@
 <wire x1="60.96" y1="81.28" x2="53.34" y2="81.28" width="0.1524" layer="91"/>
 <junction x="60.96" y="81.28"/>
-<pinref part="R7" gate="G$1" pin="1"/>
-<wire x1="53.34" y1="81.28" x2="38.1" y2="81.28" width="0.1524" layer="91"/>
 <junction x="53.34" y="81.28"/>
-<pinref part="R8" gate="G$1" pin="1"/>
-<wire x1="38.1" y1="81.28" x2="30.48" y2="81.28" width="0.1524" layer="91"/>
-<junction x="38.1" y="81.28"/>
 <pinref part="R6" gate="G$1" pin="1"/>
-<wire x1="30.48" y1="81.28" x2="22.86" y2="81.28" width="0.1524" layer="91"/>
-<junction x="30.48" y="81.28"/>
+<wire x1="53.34" y1="81.28" x2="22.86" y2="81.28" width="0.1524" layer="91"/>
 <wire x1="76.2" y1="81.28" x2="68.58" y2="81.28" width="0.1524" layer="91"/>
 </segment>
@@
 </segment>
 <segment>
-<pinref part="TXD" gate="G$1" pin="A"/>
-<wire x1="30.48" y1="101.6" x2="30.48" y2="111.76" width="0.1524" layer="91"/>
-<label x="30.48" y="111.76" size="1.778" layer="95" rot="R90"/>
-</segment>
-<segment>
 <pinref part="J1" gate="G$1" pin="3"/>
 <wire x1="124.46" y1="172.72" x2="119.38" y2="172.72" width="0.1524" layer="91"/>
@@
 <wire x1="60.96" y1="172.72" x2="78.74" y2="172.72" width="0.1524" layer="91"/>
 <label x="78.74" y="172.72" size="1.778" layer="95" xref="yes"/>
-</segment>
-<segment>
-<pinref part="RXD" gate="G$1" pin="A"/>
-<wire x1="38.1" y1="101.6" x2="38.1" y2="111.76" width="0.1524" layer="91"/>
-<label x="38.1" y="111.76" size="1.778" layer="95" rot="R90"/>
 </segment>
 <segment>
@@
 <wire x1="109.22" y1="109.22" x2="53.34" y2="109.22" width="0.1524" layer="91"/>
 <wire x1="53.34" y1="109.22" x2="53.34" y2="101.6" width="0.1524" layer="91"/>
-</segment>
-</net>
-<net name="N$10" class="0">
-<segment>
-<pinref part="RXD" gate="G$1" pin="C"/>
-<pinref part="R7" gate="G$1" pin="2"/>
-<wire x1="38.1" y1="93.98" x2="38.1" y2="91.44" width="0.1524" layer="91"/>
-</segment>
-</net>
-<net name="N$11" class="0">
-<segment>
-<pinref part="TXD" gate="G$1" pin="C"/>
-<pinref part="R8" gate="G$1" pin="2"/>
-<wire x1="30.48" y1="93.98" x2="30.48" y2="91.44" width="0.1524" layer="91"/>
 </segment>
 </net>
@@
 <compatibility>
 <note version="8.2" severity="warning">
-Since Version 8.2, Eagle supports online libraries. The ids
+Since Version 8.2, EAGLE supports online libraries. The ids
 of those online libraries will not be understood (or retained)
 with this version.

Commit message: - updated board and schematic
Parts:
- removed J2: (no value), SparkFun-Connectors:CONN_04POLAR
- removed RST: SPST, SparkFun-Switches:MOMENTARY-SWITCH-SPST-PTH-6.0MM
- removed TP1, TP2: TEST-POINT2, SparkFun-Connectors:TEST-POINT2
- removed TP10, TP11, TP12, TP13, TP14, TP15, TP16, TP5, TP6, TP7, TP8, TP9: TEST-POINTTP_15TH_THRU, SparkFun-Connectors:TEST-POINTTP_15TH_THRU
- removed TP17: MISO, SparkFun-Connectors:TEST-POINTTP_15TH_THRU
- removed TP18: MOSI, SparkFun-Connectors:TEST-POINTTP_15TH_THRU
- removed TP19: SCK, SparkFun-Connectors:TEST-POINTTP_15TH_THRU
- removed TP20: SS, SparkFun-Connectors:TEST-POINTTP_15TH_THRU
- removed TP3: SWD_CLK, SparkFun-Connectors:TEST-POINTTP_15TH_THRU
- removed TP4: SWD_SIO, SparkFun-Connectors:TEST-POINTTP_15TH_THRU
- added PROG: (no value), DC_LOAD_AU:PINHD-1X4
Connections:
- removed net /SSEL: TP20.1, U$1./SPIS_CS
- removed net MISO: TP17.1, U$1.SPIS_MISO
- removed net MOSI: TP18.1, U$1.SPIS_MOSI
- removed net N$13: TP5.1, U$1.GPIO_8
- removed net N$14: TP4.1, U$1.SWD_DIO
- removed net N$15: TP6.1, U$1.GPIO_9
- removed net N$16: TP7.1, U$1.GPIO_10
- removed net N$17: TP8.1, U$1.GPIO_12
- removed net N$18: TP9.1, U$1.GPIO_13
- removed net N$19: TP10.1, U$1.GPIO_14
- removed net N$20: TP11.1, U$1.GPIO_15
- removed net N$21: TP12.1, U$1.GPIO_22
- removed net N$22: TP13.1, U$1.GPIO_23
- removed net N$23: TP14.1, U$1.GPIO_27
- removed net N$24: TP15.1, U$1.GPIO_30
- removed net N$25: TP16.1, U$1.GPIO_31
- removed net N$5: TP3.1, U$1.SWD_CLK
- removed net SCK: TP19.1, U$1.SPIS_CLK
- new net SWD_CLK: PROG.2, U$1.SWD_CLK
- new net SWD_SIO: PROG.3, U$1.SWD_DIO
- net /RESET: no longer RST.2
- net GND: now also PROG.4; no longer J2.1, RESET.1, TP2.1
- net RXD: no longer J2.3
- net TXD: no longer J2.2
- net VCC: now also PROG.1, RESET.1; no longer J2.4, RST.1, TP1.1
Other:
- moved on the sheet: RESET
